Commit message: updated

File: urdf/Fish_HPURV_macro.urdf.xacro (robot description, xacro)
@@ -56,4 +56,5 @@
     <!-- ✅ Define Joints -->
     <joint name="${prefix}Revolute_2" type="revolute">
+      <origin xyz="-0.082983 -0.047057 0.139" rpy="0 0 0"/>
       <parent link="${prefix}base_link"/>
       <child link="${prefix}Pectal_left"/>
@@ -62,4 +63,5 @@
     </joint>
     <joint name="${prefix}Revolute_7" type="revolute">
+      <origin xyz="-0.082983 -0.047057 -0.14" rpy="0 0 0"/>
       <parent link="${prefix}base_link"/>
       <child link="${prefix}Pectal_right"/>
@@ -68,5 +70,5 @@
     </joint>
     <joint name="${prefix}Revolute_8" type="revolute">
-      <origin xyz="0.05 0 0" rpy="0 0 0"/>
+      <origin xyz="0.392742 -0.028093 0.0" rpy="0 0 0"/>
       <parent link="${prefix}base_link"/>
       <child link="${prefix}Caudal_Fin"/>
