Commit message: updated

File: urdf/fish_hpurv_macro.urdf.xacro (robot description, xacro)
@@ -17,5 +17,5 @@
         <origin xyz="0 0 0" rpy="0 0 0"/>
         <geometry>
-          <mesh filename="package://fish_hpurv_description/meshes/base_link.stl" scale="0.001 0.001 0.001"/>
+          <mesh filename="package://fish_hpurv_description/meshes/base_link.stl" scale="1 1 1"/>
         </geometry>
         <material name="fish_hpurv_silver"/>
@@ -24,14 +24,13 @@
         <origin xyz="0 0 0" rpy="0 0 0"/>
         <geometry>
-          <mesh filename="package://fish_hpurv_description/meshes/base_link.stl" scale="0.001 0.001 0.001"/>
+          <mesh filename="package://fish_hpurv_description/meshes/base_link.stl" scale="1 1 1"/>
         </geometry>
       </collision>
     </link>
-    <link name="dummy_link"/>
     <!-- Define Fins -->
     <link name="${prefix}pectal_left">
       <visual>
         <geometry>
-          <mesh filename="package://fish_hpurv_description/meshes/pectal_left.stl" scale="0.001 0.001 0.001"/>
+          <mesh filename="package://fish_hpurv_description/meshes/Pectal_left.stl" scale="1 1 1"/>
         </geometry>
       </visual>
@@ -40,5 +39,5 @@
       <visual>
         <geometry>
-          <mesh filename="package://fish_hpurv_description/meshes/pectal_right.stl" scale="0.001 0.001 0.001"/>
+          <mesh filename="package://fish_hpurv_description/meshes/Pectal_right.stl" scale="1 1 1"/>
         </geometry>
       </visual>
@@ -47,5 +46,5 @@
       <visual>
         <geometry>
-          <mesh filename="package://fish_hpurv_description/meshes/caudal_fin.stl" scale="0.001 0.001 0.001"/>
+          <mesh filename="package://fish_hpurv_description/meshes/Caudal_Fin.stl" scale="1 1 1"/>
         </geometry>
       </visual>
@@ -63,11 +62,6 @@
       <parent link="${prefix}base_link"/>
       <child link="${prefix}pectal_right"/>
-      <axis xyz="0.0 0.0 -1.0"/>
+      <axis xyz="1.0 0.0 0.0"/>
       <limit upper="0.785398" lower="-0.785398" effort="100" velocity="100"/>
-    </joint>
-    <joint name="dummy_to_base" type="fixed">
-      <parent link="dummy_link"/>
-      <child link="base_link"/>
-      <origin xyz="0 0 0" rpy="0 0 0"/>
     </joint>
     <joint name="${prefix}revolute_8" type="revolute">

Commit message: Initial commit of differential drive robot package

File: urdf/fish_hpurv_macro.urdf.xacro (robot description, xacro)
@@ -1,103 +1,71 @@
-<?xml version="1.0"?>
-<robot name="fish_hpurv" xmlns:xacro="http://www.ros.org/wiki/xacro">
-  <!-- Define Material Properties -->
-  <material name="fish_hpurv_silver">
-    <color rgba="0.700 0.700 0.700 1.000"/>
-  </material>
-  <!-- Define Main Robot Body -->
-  <xacro:macro name="fish_hpurv" params="prefix">
-    <!-- Base Link -->
-    <link name="${prefix}base_link">
-      <inertial>
-        <origin xyz="0 0 0" rpy="0 0 0"/>
-        <mass value="5.0"/>
-        <inertia ixx="0.01" iyy="0.01" izz="0.01" ixy="0" iyz="0" ixz="0"/>
-      </inertial>
-      <visual>
-        <origin xyz="0 0 0" rpy="0 0 0"/>
-        <geometry>
-          <mesh filename="package://fish_hpurv_description/meshes/base_link.stl" scale="1 1 1"/>
-        </geometry>
-        <material name="fish_hpurv_silver"/>
-      </visual>
-      <collision>
-        <origin xyz="0 0 0" rpy="0 0 0"/>
-        <geometry>
-          <mesh filename="package://fish_hpurv_description/meshes/base_link.stl" scale="1 1 1"/>
-        </geometry>
-      </collision>
-    </link>
-    <!-- Define Fins -->
-    <link name="${prefix}pectal_left">
-      <visual>
-        <geometry>
-          <mesh filename="package://fish_hpurv_description/meshes/Pectal_left.stl" scale="1 1 1"/>
-        </geometry>
-      </visual>
-    </link>
-    <link name="${prefix}pectal_right">
-      <visual>
-        <geometry>
-          <mesh filename="package://fish_hpurv_description/meshes/Pectal_right.stl" scale="1 1 1"/>
-        </geometry>
-      </visual>
-    </link>
-    <link name="${prefix}caudal_fin">
-      <visual>
-        <geometry>
-          <mesh filename="package://fish_hpurv_description/meshes/Caudal_Fin.stl" scale="1 1 1"/>
-        </geometry>
-      </visual>
-    </link>
-    <!-- Define Joints -->
-    <joint name="${prefix}revolute_2" type="revolute">
-      <origin xyz="-0.082983 -0.047057 0.139" rpy="0 0 0"/>
-      <parent link="${prefix}base_link"/>
-      <child link="${prefix}pectal_left"/>
-      <axis xyz="1.0 0.0 0.0"/>
-      <limit upper="0.785398" lower="-0.785398" effort="100" velocity="100"/>
-    </joint>
-    <joint name="${prefix}revolute_7" type="revolute">
-      <origin xyz="-0.082983 -0.047057 -0.14" rpy="0 0 0"/>
-      <parent link="${prefix}base_link"/>
-      <child link="${prefix}pectal_right"/>
-      <axis xyz="1.0 0.0 0.0"/>
-      <limit upper="0.785398" lower="-0.785398" effort="100" velocity="100"/>
-    </joint>
-    <joint name="${prefix}revolute_8" type="revolute">
-      <origin xyz="0.392742 -0.028093 0.0" rpy="0 0 0"/>
-      <parent link="${prefix}base_link"/>
-      <child link="${prefix}caudal_fin"/>
-      <axis xyz="-0.173648 0.984808 0.0"/>
-      <limit upper="0.785398" lower="-0.785398" effort="100" velocity="100"/>
-    </joint>
-    <!-- Add Gazebo Properties for Links -->
-    <gazebo reference="${prefix}base_link">
-      <material>Gazebo/Silver</material>
-      <mu1>0.2</mu1>
-      <mu2>0.2</mu2>
-      <self_collide>true</self_collide>
-      <gravity>true</gravity>
-    </gazebo>
-    <gazebo reference="${prefix}pectal_left">
-      <material>Gazebo/Silver</material>
-      <mu1>0.2</mu1>
-      <mu2>0.2</mu2>
-      <self_collide>true</self_collide>
-    </gazebo>
-    <gazebo reference="${prefix}pectal_right">
-      <material>Gazebo/Silver</material>
-      <mu1>0.2</mu1>
-      <mu2>0.2</mu2>
-      <self_collide>true</self_collide>
-    </gazebo>
-    <gazebo reference="${prefix}caudal_fin">
-      <material>Gazebo/Silver</material>
-      <mu1>0.2</mu1>
-      <mu2>0.2</mu2>
-      <self_collide>true</self_collide>
-    </gazebo>
-  </xacro:macro>
-  <!-- Instantiate the Robot -->
-  <xacro:fish_hpurv prefix=""/>
+<?xml version="1.0" ?>
+<!-- Generated using onshape-to-robot -->
+<!-- Onshape document_id: 4836a8ecee0138adbd06e5d4 / workspace_id: a33d52e229ba318a84bbb324 -->
+<robot name="fish_hpurv">
+  <!-- Link link_link1 -->
+  <link name="link_link1">
+    <inertial>
+      <origin xyz="0 0 0" rpy="0 0 0"/>
+      <mass value="0.2"/>
+      <inertia ixx="0.005" ixy="0" ixz="0" iyy="0.005" iyz="0" izz="0.005"/>
+    </inertial>
+    <visual>
+      <origin xyz="0.0228213 0.0461472 0.010826" rpy="0 0 0"/>
+      <geometry>
+        <mesh filename="package://fish_hpurv/meshes/link_link1.stl">
+          <scale>4 4 4</scale>
+        </mesh>
+      </geometry>
+      <material name="link_link1_material">
+        <color rgba="0.615686 0.811765 0.929412 1.0"/>
+      </material>
+    </visual>
+    <collision>
+      <origin xyz="0.0228213 0.0461472 0.010826" rpy="0 0 0"/>
+      <geometry>
+        <mesh filename="package://fish_hpurv/meshes/link_link1.stl">
+          <scale>4 4 4</scale>
+        </mesh>
+      </geometry>
+    </collision>
+  </link>
+  <!-- Link link_link2 -->
+  <link name="link_link2">
+    <inertial>
+      <origin xyz="0 0 0" rpy="0 0 0"/>
+      <mass value="0.1"/>
+      <inertia ixx="0.001" ixy="0" ixz="0" iyy="0.001" iyz="0" izz="0.001"/>
+    </inertial>
+    <visual>
+      <origin xyz="0 0 0" rpy="3.14159 0 0"/>
+      <geometry>
+        <mesh filename="package://fish_hpurv/meshes/link_link2.stl">
+          <scale>4 4 4</scale>
+        </mesh>
+      </geometry>
+      <material name="link_link2_material">
+        <color rgba="0.615686 0.811765 0.929412 1.0"/>
+      </material>
+    </visual>
+    <collision>
+      <origin xyz="0 0 0" rpy="3.14159 0 0"/>
+      <geometry>
+        <mesh filename="package://fish_hpurv/meshes/link_link2.stl">
+          <scale>4 4 4</scale>
+        </mesh>
+      </geometry>
+    </collision>
+  </link>
+  <!-- Joint from link_link1 to link_link2 -->
+  <joint name="join1" type="prismatic">
+    <origin xyz="0.0228213 0.0461472 0.035826" rpy="3.14159 0 0"/>
+    <parent link="link_link1"/>
+    <child link="link_link2"/>
+    <axis xyz="0 0 1"/>
+    <limit effort="10" velocity="10" lower="-1" upper="1"/>
+  </joint>
+  <!-- Mark the robot as static so it won't fall -->
+  <gazebo>
+    <static>true</static>
+  </gazebo>
 </robot>

Commit message: Exclude models directory from tracking in fish_hpurv package

File: urdf/fish_hpurv_macro.urdf.xacro (robot description, xacro)
@@ -1,71 +1,229 @@
-<?xml version="1.0" ?>
-<!-- Generated using onshape-to-robot -->
-<!-- Onshape document_id: 4836a8ecee0138adbd06e5d4 / workspace_id: a33d52e229ba318a84bbb324 -->
-<robot name="fish_hpurv">
-  <!-- Link link_link1 -->
-  <link name="link_link1">
-    <inertial>
-      <origin xyz="0 0 0" rpy="0 0 0"/>
-      <mass value="0.2"/>
-      <inertia ixx="0.005" ixy="0" ixz="0" iyy="0.005" iyz="0" izz="0.005"/>
-    </inertial>
-    <visual>
-      <origin xyz="0.0228213 0.0461472 0.010826" rpy="0 0 0"/>
-      <geometry>
-        <mesh filename="package://fish_hpurv/meshes/link_link1.stl">
-          <scale>4 4 4</scale>
-        </mesh>
-      </geometry>
-      <material name="link_link1_material">
-        <color rgba="0.615686 0.811765 0.929412 1.0"/>
-      </material>
-    </visual>
-    <collision>
-      <origin xyz="0.0228213 0.0461472 0.010826" rpy="0 0 0"/>
-      <geometry>
-        <mesh filename="package://fish_hpurv/meshes/link_link1.stl">
-          <scale>4 4 4</scale>
-        </mesh>
-      </geometry>
-    </collision>
-  </link>
-  <!-- Link link_link2 -->
-  <link name="link_link2">
-    <inertial>
-      <origin xyz="0 0 0" rpy="0 0 0"/>
-      <mass value="0.1"/>
-      <inertia ixx="0.001" ixy="0" ixz="0" iyy="0.001" iyz="0" izz="0.001"/>
-    </inertial>
-    <visual>
-      <origin xyz="0 0 0" rpy="3.14159 0 0"/>
-      <geometry>
-        <mesh filename="package://fish_hpurv/meshes/link_link2.stl">
-          <scale>4 4 4</scale>
-        </mesh>
-      </geometry>
-      <material name="link_link2_material">
-        <color rgba="0.615686 0.811765 0.929412 1.0"/>
-      </material>
-    </visual>
-    <collision>
-      <origin xyz="0 0 0" rpy="3.14159 0 0"/>
-      <geometry>
-        <mesh filename="package://fish_hpurv/meshes/link_link2.stl">
-          <scale>4 4 4</scale>
-        </mesh>
-      </geometry>
-    </collision>
-  </link>
-  <!-- Joint from link_link1 to link_link2 -->
-  <joint name="join1" type="prismatic">
-    <origin xyz="0.0228213 0.0461472 0.035826" rpy="3.14159 0 0"/>
-    <parent link="link_link1"/>
-    <child link="link_link2"/>
-    <axis xyz="0 0 1"/>
-    <limit effort="10" velocity="10" lower="-1" upper="1"/>
-  </joint>
-  <!-- Mark the robot as static so it won't fall -->
-  <gazebo>
-    <static>true</static>
-  </gazebo>
-</robot>
+<sdf version="1.6">
+  <model name="fish_hpurv">
+    <!-- Base Link: link_base -->
+    <link name="link_base">
+      <!-- The link frame is set at the origin -->
+      <pose>0 0 0 0 0 0</pose>
+      <inertial>
+        <!-- Move the URDF inertial offset into the link's frame by zeroing the inertial pose -->
+        <pose>0 0 0 0 0 0</pose>
+        <mass>50</mass>
+        <inertia>
+          <ixx>0.01</ixx>
+          <ixy>0</ixy>
+          <ixz>0</ixz>
+          <iyy>0.01</iyy>
+          <iyz>0</iyz>
+          <izz>0.01</izz>
+        </inertia>
+      </inertial>
+      <collision name="link_base_collision">
+        <!-- Element pose zeroed; the mesh should be positioned relative to the link frame -->
+        <pose>0 0 0 0 0 0</pose>
+        <geometry>
+          <mesh>
+            <scale>1 1 1</scale>
+            <uri>model://fish_hpurv/meshes/link_base.stl</uri>
+          </mesh>
+        </geometry>
+      </collision>
+      <visual name="link_base_visual">
+        <pose>0 0 0 0 0 0</pose>
+        <geometry>
+          <mesh>
+            <scale>1 1 1</scale>
+            <uri>model://fish_hpurv/meshes/link_base.stl</uri>
+          </mesh>
+        </geometry>
+      </visual>
+    </link>
+    <!-- Joint: caudal_joint -->
+    <joint name="caudal_joint" type="revolute">
+      <!-- Use the URDF joint origin directly as the transformation from link_base frame to link_caudal frame -->
+      <pose>0.425323 0.0803079 -0.0204279 -1.5708 0 0</pose>
+      <parent>link_base</parent>
+      <child>link_caudal</child>
+      <axis>
+        <xyz>0 0 1</xyz>
+        <limit>
+          <lower>-0.523599</lower>
+          <upper>0.523599</upper>
+          <effort>10</effort>
+          <velocity>10</velocity>
+        </limit>
+        <dynamics>
+          <damping>1.5</damping>
+          <spring_reference>0</spring_reference>
+          <spring_stiffness>0</spring_stiffness>
+        </dynamics>
+      </axis>
+    </joint>
+    <!-- Child Link: link_caudal -->
+    <link name="link_caudal">
+      <!-- The link frame is now at the joint origin -->
+      <pose>0 0 0 0 0 0</pose>
+      <inertial>
+        <!-- The inertial offset from URDF is applied relative to the link frame -->
+        <pose>-0.378805 0 -0.05 1.5708 0 0</pose>
+        <mass>10</mass>
+        <inertia>
+          <ixx>0.005</ixx>
+          <ixy>0</ixy>
+          <ixz>0</ixz>
+          <iyy>0.005</iyy>
+          <iyz>0</iyz>
+          <izz>0.005</izz>
+        </inertia>
+      </inertial>
+      <collision name="link_caudal_collision">
+        <pose>0 0 0 0 0 0</pose>
+        <geometry>
+          <mesh>
+            <scale>1 1 1</scale>
+            <uri>model://fish_hpurv/meshes/link_caudal.stl</uri>
+          </mesh>
+        </geometry>
+      </collision>
+      <visual name="link_caudal_visual">
+        <pose>0 0 0 0 0 0</pose>
+        <geometry>
+          <mesh>
+            <scale>1 1 1</scale>
+            <uri>model://fish_hpurv/meshes/link_caudal.stl</uri>
+          </mesh>
+        </geometry>
+      </visual>
+    </link>
+    <!-- Joint: joint1 (for left pectoral fin) -->
+    <joint name="joint1" type="revolute">
+      <pose>-0.0504018 0.00224307 0.118572 3.14159 0 0</pose>
+      <parent>link_base</parent>
+      <child>link_pectoral_left</child>
+      <axis>
+        <xyz>0 0 1</xyz>
+        <limit>
+          <lower>-0.785398</lower>
+          <upper>0.785398</upper>
+          <effort>10</effort>
+          <velocity>10</velocity>
+        </limit>
+        <dynamics>
+          <damping>1.5</damping>
+          <spring_reference>0</spring_reference>
+          <spring_stiffness>0</spring_stiffness>
+        </dynamics>
+      </axis>
+    </joint>
+    <!-- Child Link: link_pectoral_left -->
+    <link name="link_pectoral_left">
+      <!-- The link frame is at the joint origin -->
+      <pose>0 0 0 0 0 0</pose>
+      <inertial>
+        <!-- Apply the URDF offset for this fin -->
+        <pose>0.0829833 -0.0470575 0.13 3.14159 0 0</pose>
+        <mass>5</mass>
+        <inertia>
+          <ixx>0.001</ixx>
+          <ixy>0</ixy>
+          <ixz>0</ixz>
+          <iyy>0.001</iyy>
+          <iyz>0</iyz>
+          <izz>0.001</izz>
+        </inertia>
+      </inertial>
+      <collision name="link_pectoral_left_collision">
+        <pose>0 0 0 0 0 0</pose>
+        <geometry>
+          <mesh>
+            <scale>1 1 1</scale>
+            <uri>model://fish_hpurv/meshes/link_pectoral_left.stl</uri>
+          </mesh>
+        </geometry>
+      </collision>
+      <visual name="link_pectoral_left_visual">
+        <pose>0 0 0 0 0 0</pose>
+        <geometry>
+          <mesh>
+            <scale>1 1 1</scale>
+            <uri>model://fish_hpurv/meshes/link_pectoral_left.stl</uri>
+          </mesh>
+        </geometry>
+      </visual>
+    </link>
+    <!-- Joint: joint2 (for right pectoral fin) -->
+    <joint name="joint2" type="revolute">
+      <pose>-0.0504018 0.00224307 -0.160428 0 0 0</pose>
+      <parent>link_base</parent>
+      <child>link_pectoral_right</child>
+      <axis>
+        <xyz>0 0 1</xyz>
+        <limit>
+          <lower>-0.785398</lower>
+          <upper>0.785398</upper>
+          <effort>10</effort>
+          <velocity>10</velocity>
+        </limit>
+        <dynamics>
+          <damping>1.5</damping>
+          <spring_reference>0</spring_reference>
+          <spring_stiffness>0</spring_stiffness>
+        </dynamics>
+      </axis>
+    </joint>
+    <!-- Child Link: link_pectoral_right -->
+    <link name="link_pectoral_right">
+      <!-- The link frame is at the joint origin -->
+      <pose>0 0 0 0 0 0</pose>
+      <inertial>
+        <pose>0.0829833 0.0470575 0.13 0 0 0</pose>
+        <mass>5</mass>
+        <inertia>
+          <ixx>0.001</ixx>
+          <ixy>0</ixy>
+          <ixz>0</ixz>
+          <iyy>0.001</iyy>
+          <iyz>0</iyz>
+          <izz>0.001</izz>
+        </inertia>
+      </inertial>
+      <collision name="link_pectoral_right_collision">
+        <pose>0 0 0 0 0 0</pose>
+        <geometry>
+          <mesh>
+            <scale>1 1 1</scale>
+            <uri>model://fish_hpurv/meshes/link_pectoral_right.stl</uri>
+          </mesh>
+        </geometry>
+      </collision>
+      <visual name="link_pectoral_right_visual">
+        <pose>0 0 0 0 0 0</pose>
+        <geometry>
+          <mesh>
+            <scale>1 1 1</scale>
+            <uri>model://fish_hpurv/meshes/link_pectoral_right.stl</uri>
+          </mesh>
+        </geometry>
+      </visual>
+    </link>
+    <!-- GAZEBO PLUGIN: Buoyancy -->
+    <plugin name="buoyancy_plugin" filename="libBuoyancyPlugin.so">
+      <fluid_density>1000</fluid_density>
+      <link name="link_base">
+        <volume>0.05</volume>
+        <center_of_volume>0.0325815 0.0493006 -0.0204279</center_of_volume>
+      </link>
+      <link name="link_caudal">
+        <volume>0.01</volume>
+        <center_of_volume>-0.378805 0 -0.05</center_of_volume>
+      </link>
+      <link name="link_pectoral_left">
+        <volume>0.005</volume>
+        <center_of_volume>0.0829833 -0.0470575 0.13</center_of_volume>
+      </link>
+      <link name="link_pectoral_right">
+        <volume>0.005</volume>
+        <center_of_volume>0.0829833 0.0470575 0.13</center_of_volume>
+      </link>
+    </plugin>
+  </model>
+</sdf>
