Commit message: updated

File: urdf/fish_hpurv_macro.urdf.xacro (robot description, xacro)
@@ -1,5 +1,3 @@
-<?xml version="1.0" ?>
-<robot name="fish_hpurv">
-  <!-- Link: link_base -->
+<robot name="fish_hpurv" xmlns:xacro="http://www.ros.org/wiki/xacro">
   <link name="link_base">
     <inertial>
@@ -24,13 +22,12 @@
     </collision>
   </link>
-  <!-- Link: link_caudal -->
   <link name="link_caudal">
     <inertial>
-      <origin xyz="-0.378805 2.04697e-16 -0.05" rpy="0 0 0"/>
+      <origin xyz="-0.378805 0 -0.05" rpy="1.5708 0 0"/>
       <mass value="0.2"/>
       <inertia ixx="0.005" ixy="0" ixz="0" iyy="0.005" iyz="0" izz="0.005"/>
     </inertial>
     <visual>
-      <origin xyz="-0.378805 2.04697e-16 -0.05" rpy="0 0 0"/>
+      <origin xyz="-0.378805 0 -0.05" rpy="1.5708 0 0"/>
       <geometry>
         <mesh filename="$(find fish_hpurv)/meshes/link_caudal.stl"/>
@@ -41,5 +38,5 @@
     </visual>
     <collision>
-      <origin xyz="-0.378805 2.04697e-16 -0.05" rpy="0 0 0"/>
+      <origin xyz="-0.378805 0 -0.05" rpy="1.5708 0 0"/>
       <geometry>
         <mesh filename="$(find fish_hpurv)/meshes/link_caudal.stl"/>
@@ -47,7 +44,6 @@
     </collision>
   </link>
-  <!-- Joint: caudal_joint (from link_base to link_caudal) -->
   <joint name="caudal_joint" type="revolute">
-    <origin xyz="0.425323 0.0953079 0.02" rpy="-1.5708 0 0"/>
+    <origin xyz="0.425323 0.05 0.06" rpy="0 0 0"/>
     <parent link="link_base"/>
     <child link="link_caudal"/>
@@ -55,13 +51,12 @@
     <limit effort="10" velocity="10" lower="-0.523599" upper="0.523599"/>
   </joint>
-  <!-- Link: link_pectoral_left -->
   <link name="link_pectoral_left">
     <inertial>
-      <origin xyz="0.0829833 -0.0470575 0.13" rpy="1.5708 0 0"/>
+      <origin xyz="0.0829833 -0.0470575 0.13" rpy="3.14 0 0"/>
       <mass value="0.1"/>
       <inertia ixx="0.001" ixy="0" ixz="0" iyy="0.001" iyz="0" izz="0.001"/>
     </inertial>
     <visual>
-      <origin xyz="0.0829833 -0.0470575 0.13" rpy="1.5708 0 0"/>
+      <origin xyz="0.0829833 -0.0470575 0.13" rpy="3.14 0 0"/>
       <geometry>
         <mesh filename="$(find fish_hpurv)/meshes/link_pectoral_left.stl"/>
@@ -72,5 +67,5 @@
     </visual>
     <collision>
-      <origin xyz="0.0829833 -0.0470575 0.13" rpy="1.5708 0 0"/>
+      <origin xyz="0.0829833 -0.0470575 0.13" rpy="3.14 0 0"/>
       <geometry>
         <mesh filename="$(find fish_hpurv)/meshes/link_pectoral_left.stl"/>
@@ -78,7 +73,6 @@
     </collision>
   </link>
-  <!-- Joint: joint1 (from link_base to link_pectoral_left) -->
   <joint name="joint1" type="revolute">
-    <origin xyz="-0.0504018 0.00224307 0.158572" rpy="3.14159 0 0"/>
+    <origin xyz="-0.05 0.18 0.035" rpy="1.57 0 0"/>
     <parent link="link_base"/>
     <child link="link_pectoral_left"/>
@@ -86,13 +80,12 @@
     <limit effort="10" velocity="10" lower="-0.785398" upper="0.785398"/>
   </joint>
-  <!-- Link: link_pectoral_right -->
   <link name="link_pectoral_right">
     <inertial>
-      <origin xyz="0.0829833 0.0470575 0.13" rpy="-1.5708 0 0"/>
+      <origin xyz="0.0829833 0.0470575 0.13" rpy="0 0 0"/>
       <mass value="0.1"/>
       <inertia ixx="0.001" ixy="0" ixz="0" iyy="0.001" iyz="0" izz="0.001"/>
     </inertial>
     <visual>
-      <origin xyz="0.0829833 0.0470575 0.13" rpy="-1.5708 0 0"/>
+      <origin xyz="0.0829833 0.0470575 0.13" rpy="0 0 0"/>
       <geometry>
         <mesh filename="$(find fish_hpurv)/meshes/link_pectoral_right.stl"/>
@@ -103,5 +96,5 @@
     </visual>
     <collision>
-      <origin xyz="0.0829833 0.0470575 0.13" rpy="-1.5708 0 0"/>
+      <origin xyz="0.0829833 0.0470575 0.13" rpy="0 0 0"/>
       <geometry>
         <mesh filename="$(find fish_hpurv)/meshes/link_pectoral_right.stl"/>
@@ -109,7 +102,6 @@
     </collision>
   </link>
-  <!-- Joint: joint2 (from link_base to link_pectoral_right) -->
   <joint name="joint2" type="revolute">
-    <origin xyz="-0.0504018 0.00224307 -0.120328" rpy="0 0 0"/>
+    <origin xyz="-0.05 -0.08 0.035" rpy="-1.57 0 0"/>
     <parent link="link_base"/>
     <child link="link_pectoral_right"/>
@@ -120,10 +112,8 @@
     <parent link="link_base"/>
     <child link="laser_frame"/>
-    <!-- Place the sensor slightly ahead; here we use an offset relative to link_base -->
     <origin xyz="0.0325815 0.0493006 0.02" rpy="0 0 0"/>
   </joint>
   <link name="laser_frame">
     <inertial>
-      <!-- The inertial origin is at (0,0,0) for the laser_frame -->
       <origin xyz="0 0 0" rpy="0 0 0"/>
       <mass value="0.1"/>
@@ -146,5 +136,4 @@
     </collision>
   </link>
-  <!-- Sensor plugin for the LiDAR remains as before -->
   <gazebo reference="laser_frame">
     <material>Gazebo/Red</material>
@@ -178,10 +167,8 @@
     <parent link="link_base"/>
     <child link="imu_link"/>
-    <!-- Place the IMU at a chosen offset on link_base; adjust xyz as needed -->
     <origin xyz="0.0325815 0.0493006 0.02" rpy="0 0 0"/>
   </joint>
   <link name="imu_link">
     <inertial>
-      <!-- Small inertial values for the sensor -->
       <origin xyz="0 0 0" rpy="0 0 0"/>
       <mass value="0.1"/>
@@ -218,40 +205,33 @@
     </sensor>
   </gazebo>
-<gazebo reference="link_base">
-  <sensor name="dvl_sensor" type="ray">
-    <!-- Sensor pose relative to link_base (positioned 1.5708 radians (90°) downward) -->
-    <pose>0.03 -0.085 -0.06  0  3.14 0</pose>
-    <visualize>true</visualize>
-    <update_rate>10</update_rate>
-    <ray>
-      <scan>
-        <horizontal>
-          <!-- 4 beams spanning 360° -->
-          <samples>4</samples>
-          <min_angle>0</min_angle>
-          <max_angle>6.28319</max_angle> <!-- 360° -->
-        </horizontal>
-        <vertical>
-          <!-- Tilt beams 70° from sensor's horizontal plane (20° from vertical) -->
-          <samples>1</samples>
-          <min_angle>1.2217</min_angle> <!-- 70° in radians -->
-          <max_angle>1.2217</max_angle>
-        </vertical>
-      </scan>
-      <range>
-        <min>0.1</min>
-        <max>100</max>
-      </range>
-    </ray>
-    <plugin name="custom_dvl_plugin" filename="libfish_dvl_plugin.so"/>
-  </sensor>
-</gazebo>
+  <gazebo reference="link_base">
+    <sensor name="dvl_sensor" type="ray">
+      <pose>0.03 -0.085 -0.06  0  3.14 0</pose>
+      <visualize>true</visualize>
+      <update_rate>10</update_rate>
+      <ray>
+        <scan>
+          <horizontal>
+            <samples>4</samples>
+            <min_angle>0</min_angle>
+            <max_angle>6.28319</max_angle>
+          </horizontal>
+          <vertical>
+            <samples>1</samples>
+            <min_angle>1.2217</min_angle>
+            <max_angle>1.2217</max_angle>
+          </vertical>
+        </scan>
+        <range>
+          <min>0.1</min>
+          <max>100</max>
+        </range>
+      </ray>
+      <plugin name="custom_dvl_plugin" filename="libfish_dvl_plugin.so"/>
+    </sensor>
+  </gazebo>
   <gazebo>
-    <!-- Buoyancy Plugin: Merge laser_frame into link_base -->
     <plugin name="buoyancy_plugin" filename="libBuoyancyPlugin.so">
       <fluid_density>1000</fluid_density>
-      <!-- For link_base, add the mass/volume of the laser_frame -->
-      <!-- Original link_base volume: 0.012; add 0.0001 from laser_frame = 0.0121 -->
-      <!-- The center of volume for link_base remains essentially unchanged -->
       <link name="link_base">
         <volume>0.0122</volume>
@@ -260,5 +240,5 @@
       <link name="link_caudal">
         <volume>0.0002</volume>
-        <center_of_volume>-0.378805 0  -0.05</center_of_volume>
+        <center_of_volume>-0.378805 0 -0.05</center_of_volume>
       </link>
       <link name="link_pectoral_left">
@@ -270,29 +250,29 @@
         <center_of_volume>0.0829833 0.0470575 0.13</center_of_volume>
       </link>
-      <!-- Remove the separate laser_frame entry so that its mass/volume is merged with link_base -->
     </plugin>
-    <plugin name="hydrodynamics_plugin" filename="libHydrodynamicsPlugin.so">
-      <!-- Added mass terms (example values) -->
-      <xDotU>-10.0</xDotU>
-      <yDotV>-10.0</yDotV>
-      <zDotW>-10.0</zDotW>
-      <kDotP>-0.1</kDotP>
-      <mDotQ>-0.1</mDotQ>
-      <nDotR>-0.1</nDotR>
-      <!-- Linear and quadratic damping coefficients (example values) -->
-      <xUabsU>-0.32282</xUabsU>
-      <xU>-2.5</xU>
-      <yVabsV>-0.1</yVabsV>
-      <yV>-0.5</yV>
-      <zWabsW>-0.1</zWabsW>
-      <zW>-0.5</zW>
-      <kPabsP>-0.5</kPabsP>
-      <kP>-0.5</kP>
-      <mQabsQ>-0.5</mQabsQ>
-      <mQ>-0.5</mQ>
-      <nRabsR>-0.5</nRabsR>
-      <nR>-0.5</nR>
-      <default_current>0 0 0</default_current>
+    <plugin name="gazebo_ros2_control" filename="libgazebo_ros2_control.so">
+      <robotNamespace>/</robotNamespace>
+      <parameters>$(find fish_hpurv)/config/my_controllers.yaml</parameters>
     </plugin>
   </gazebo>
+  <ros2_control name="FishSim" type="system">
+    <hardware>
+      <plugin>gazebo_ros2_control/GazeboSystem</plugin>
+    </hardware>
+    <joint name="caudal_joint">
+      <command_interface name="position"/>
+      <state_interface name="position"/>
+      <state_interface name="velocity"/>
+    </joint>
+    <joint name="joint1">
+      <command_interface name="position"/>
+      <state_interface name="position"/>
+      <state_interface name="velocity"/>
+    </joint>
+    <joint name="joint2">
+      <command_interface name="position"/>
+      <state_interface name="position"/>
+      <state_interface name="velocity"/>
+    </joint>
+  </ros2_control>
 </robot>

Commit message: updated

File: urdf/fish_hpurv_macro.urdf.xacro (robot description, xacro)
@@ -1,3 +1,6 @@
 <robot name="fish_hpurv" xmlns:xacro="http://www.ros.org/wiki/xacro">
+  <xacro:include filename="$(find uuv_descriptions)/urdf/common.urdf.xacro"/>
+  <xacro:include filename="$(find uuv_gazebo_ros_plugins)/urdf/fin_snippets.xacro"/>
+  <xacro:include filename="$(find uuv_gazebo_ros_plugins)/urdf/snippets.xacro"/>
   <link name="link_base">
     <inertial>
@@ -250,4 +253,8 @@
         <center_of_volume>0.0829833 0.0470575 0.13</center_of_volume>
       </link>
+      <link name="fish_hpurv/fin1">
+        <volume>0.0000001</volume>
+        <center_of_volume>0.0829833 0.0470575 0.13</center_of_volume>
+      </link>
     </plugin>
     <plugin name="gazebo_ros2_control" filename="libgazebo_ros2_control.so">
@@ -276,3 +283,22 @@
     </joint>
   </ros2_control>
+<xacro:fin_two_lines_macro
+    namespace="fish_hpurv"
+    parent_link="link_base"
+    fin_id="1"
+    min_joint_limit="-0.5"
+    max_joint_limit="0.5"
+    mesh_filename="$(find fish_hpurv)/meshes/fin1.stl"
+    fin_dynamics_time_constant="1.0"
+    fin_cross_section_area="0.1"
+    fluid_density="1000"
+    a0="0.0"
+    alpha_stall="15"
+    cla="0.1"
+    cla_stall="0.2"
+    cda="0.01"
+    cda_stall="0.02"
+    current_velocity_topic="/current_velocity">
+  <origin xyz="0.1 0 0" rpy="0 0 0" />
+</xacro:fin_two_lines_macro>
 </robot>
