Commit message: Update inside fish_hpurv

File: urdf/fish_hpurv_macro.urdf.xacro (robot description, xacro)
@@ -1,259 +1,105 @@
 <robot name="fish_hpurv" xmlns:xacro="http://www.ros.org/wiki/xacro">
-  <xacro:include filename="$(find uuv_descriptions)/urdf/common.urdf.xacro"/>
-  <xacro:include filename="$(find uuv_gazebo_ros_plugins)/urdf/fin_snippets.xacro"/>
-  <xacro:include filename="$(find uuv_gazebo_ros_plugins)/urdf/snippets.xacro"/>
+  <xacro:include filename="$(find uuv_descriptions)/urdf/common.urdf.xacro" />
+  <xacro:include filename="$(find uuv_gazebo_ros_plugins)/urdf/fin_snippets.xacro" />
+  <xacro:include filename="$(find uuv_gazebo_ros_plugins)/urdf/snippets.xacro" />
   <link name="link_base">
     <inertial>
-      <origin xyz="0.0325815 0.0493006 -0.0204279" rpy="1.57 0 0"/>
-      <mass value="12"/>  <!-- assume base mass remains 12 kg -->
-      <inertia ixx="0.01" ixy="0" ixz="0" iyy="0.01" iyz="0" izz="0.01"/>
+      <origin xyz="0.246461 -0.269567 0.0980965" rpy="0 -0 0"/>
+      <mass value="1" />
+      <inertia ixx="0.01" ixy="0" ixz="0" iyy="0.01" iyz="0" izz="0.01" />
     </inertial>
     <visual>
-      <origin xyz="0.0325815 0.0493006 0.02" rpy="1.57 0 0"/>
+      <origin xyz="0.246461 -0.269567 0.0980965" rpy="0 -0 0"/>
       <geometry>
-        <mesh filename="$(find fish_hpurv)/meshes/link_base.stl"/>
+        <mesh filename="$(find fish_hpurv)/meshes/link_base.stl" />
       </geometry>
       <material name="link_base_material">
-        <color rgba="0.796078 0.823529 0.937255 1.0"/>
+        <color rgba="0.796078 0.823529 0.937255 1.0" />
       </material>
     </visual>
     <collision>
-      <origin xyz="0.0325815 0.0493006 -0.0204279" rpy="1.57 0 0"/>
+      <origin xyz="0.246461 -0.269567 0.0980965" rpy="0 -0 0"/>
       <geometry>
-        <mesh filename="$(find fish_hpurv)/meshes/link_base.stl"/>
+        <mesh filename="$(find fish_hpurv)/meshes/link_base.stl" />
       </geometry>
     </collision>
   </link>
-  <link name="link_caudal">
-    <inertial>
-      <origin xyz="-0.378805 0 -0.05" rpy="1.5708 0 0"/>
-      <mass value="0.2"/>
-      <inertia ixx="0.005" ixy="0" ixz="0" iyy="0.005" iyz="0" izz="0.005"/>
-    </inertial>
-    <visual>
-      <origin xyz="-0.378805 0 -0.05" rpy="1.5708 0 0"/>
-      <geometry>
-        <mesh filename="$(find fish_hpurv)/meshes/link_caudal.stl"/>
-      </geometry>
-      <material name="link_caudal_material">
-        <color rgba="0.796078 0.823529 0.937255 1.0"/>
-      </material>
-    </visual>
-    <collision>
-      <origin xyz="-0.378805 0 -0.05" rpy="1.5708 0 0"/>
-      <geometry>
-        <mesh filename="$(find fish_hpurv)/meshes/link_caudal.stl"/>
-      </geometry>
-    </collision>
-  </link>
-  <joint name="caudal_joint" type="revolute">
-    <origin xyz="0.425323 0.05 0.06" rpy="0 0 0"/>
-    <parent link="link_base"/>
-    <child link="link_caudal"/>
-    <axis xyz="0 0 1"/>
-    <limit effort="10" velocity="10" lower="-0.523599" upper="0.523599"/>
-  </joint>
-  <link name="link_pectoral_left">
-    <inertial>
-      <origin xyz="0.0829833 -0.0470575 0.13" rpy="3.14 0 0"/>
-      <mass value="0.1"/>
-      <inertia ixx="0.001" ixy="0" ixz="0" iyy="0.001" iyz="0" izz="0.001"/>
-    </inertial>
-    <visual>
-      <origin xyz="0.0829833 -0.0470575 0.13" rpy="3.14 0 0"/>
-      <geometry>
-        <mesh filename="$(find fish_hpurv)/meshes/link_pectoral_left.stl"/>
-      </geometry>
-      <material name="link_pectoral_left_material">
-        <color rgba="0.796078 0.823529 0.937255 1.0"/>
-      </material>
-    </visual>
-    <collision>
-      <origin xyz="0.0829833 -0.0470575 0.13" rpy="3.14 0 0"/>
-      <geometry>
-        <mesh filename="$(find fish_hpurv)/meshes/link_pectoral_left.stl"/>
-      </geometry>
-    </collision>
-  </link>
-  <joint name="joint1" type="revolute">
-    <origin xyz="-0.05 0.18 0.035" rpy="1.57 0 0"/>
-    <parent link="link_base"/>
-    <child link="link_pectoral_left"/>
-    <axis xyz="0 0 1"/>
-    <limit effort="10" velocity="10" lower="-0.785398" upper="0.785398"/>
-  </joint>
-  <link name="link_pectoral_right">
-    <inertial>
-      <origin xyz="0.0829833 0.0470575 0.13" rpy="0 0 0"/>
-      <mass value="0.1"/>
-      <inertia ixx="0.001" ixy="0" ixz="0" iyy="0.001" iyz="0" izz="0.001"/>
-    </inertial>
-    <visual>
-      <origin xyz="0.0829833 0.0470575 0.13" rpy="0 0 0"/>
-      <geometry>
-        <mesh filename="$(find fish_hpurv)/meshes/link_pectoral_right.stl"/>
-      </geometry>
-      <material name="link_pectoral_right_material">
-        <color rgba="0.796078 0.823529 0.937255 1.0"/>
-      </material>
-    </visual>
-    <collision>
-      <origin xyz="0.0829833 0.0470575 0.13" rpy="0 0 0"/>
-      <geometry>
-        <mesh filename="$(find fish_hpurv)/meshes/link_pectoral_right.stl"/>
-      </geometry>
-    </collision>
-  </link>
-  <joint name="joint2" type="revolute">
-    <origin xyz="-0.05 -0.08 0.035" rpy="-1.57 0 0"/>
-    <parent link="link_base"/>
-    <child link="link_pectoral_right"/>
-    <axis xyz="0 0 1"/>
-    <limit effort="10" velocity="10" lower="-0.785398" upper="0.785398"/>
-  </joint>
-  <joint name="laser_joint" type="fixed">
-    <parent link="link_base"/>
-    <child link="laser_frame"/>
-    <origin xyz="0.0325815 0.0493006 0.02" rpy="0 0 0"/>
-  </joint>
-  <link name="laser_frame">
-    <inertial>
-      <origin xyz="0 0 0" rpy="0 0 0"/>
-      <mass value="0.1"/>
-      <inertia ixx="0.0001" ixy="0" ixz="0" iyy="0.0001" iyz="0" izz="0.0001"/>
-    </inertial>
-    <visual>
-      <origin xyz="0 0 0" rpy="0 0 0"/>
-      <geometry>
-        <cylinder radius="0.05" length="0.04"/>
-      </geometry>
-      <material name="red">
-        <color rgba="1 0 0 1"/>
-      </material>
-    </visual>
-    <collision>
-      <origin xyz="0 0 0" rpy="0 0 0"/>
-      <geometry>
-        <cylinder radius="0.05" length="0.04"/>
-      </geometry>
-    </collision>
-  </link>
-  <gazebo reference="laser_frame">
-    <material>Gazebo/Red</material>
-    <sensor name="laser" type="ray">
-      <pose>0 0 0 0 0 0</pose>
-      <visualize>true</visualize>
-      <update_rate>10</update_rate>
-      <ray>
-        <scan>
-          <horizontal>
-            <samples>360</samples>
-            <min_angle>-3.14</min_angle>
-            <max_angle>3.14</max_angle>
-          </horizontal>
-        </scan>
-        <range>
-          <min>0.3</min>
-          <max>12</max>
-        </range>
-      </ray>
-      <plugin name="laser_controller" filename="libgazebo_ros_laser.so">
-        <ros>
-          <argument>~/out:=/scan</argument>
-        </ros>
-        <output_type>sensor_msgs/LaserScan</output_type>
-        <frame_name>laser_frame</frame_name>
-      </plugin>
-    </sensor>
-  </gazebo>
-  <joint name="imu_joint" type="fixed">
-    <parent link="link_base"/>
-    <child link="imu_link"/>
-    <origin xyz="0.0325815 0.0493006 0.02" rpy="0 0 0"/>
-  </joint>
-  <link name="imu_link">
-    <inertial>
-      <origin xyz="0 0 0" rpy="0 0 0"/>
-      <mass value="0.1"/>
-      <inertia ixx="0.000001" ixy="0" ixz="0" iyy="0.000001" iyz="0" izz="0.000001"/>
-    </inertial>
-    <visual>
-      <origin xyz="0 0 0" rpy="0 0 0"/>
-      <geometry>
-        <box size="0.01 0.01 0.01"/>
-      </geometry>
-      <material name="blue">
-        <color rgba="0 0 1 1"/>
-      </material>
-    </visual>
-    <collision>
-      <origin xyz="0 0 0" rpy="0 0 0"/>
-      <geometry>
-        <box size="0.01 0.01 0.01"/>
-      </geometry>
-    </collision>
-  </link>
-  <gazebo reference="imu_link">
-    <sensor name="imu_sensor" type="imu">
-      <update_rate>50</update_rate>
-      <always_on>true</always_on>
-      <visualize>true</visualize>
-      <plugin name="imu_plugin" filename="libgazebo_ros_imu.so">
-        <ros>
-          <argument>~/out:=/imu/data</argument>
-        </ros>
-        <topicName>/imu/data</topicName>
-        <frameName>imu_link</frameName>
-      </plugin>
-    </sensor>
-  </gazebo>
-  <gazebo reference="link_base">
-    <sensor name="dvl_sensor" type="ray">
-      <pose>0.03 -0.085 -0.06  0  3.14 0</pose>
-      <visualize>true</visualize>
-      <update_rate>10</update_rate>
-      <ray>
-        <scan>
-          <horizontal>
-            <samples>4</samples>
-            <min_angle>0</min_angle>
-            <max_angle>6.28319</max_angle>
-          </horizontal>
-          <vertical>
-            <samples>1</samples>
-            <min_angle>1.2217</min_angle>
-            <max_angle>1.2217</max_angle>
-          </vertical>
-        </scan>
-        <range>
-          <min>0.1</min>
-          <max>100</max>
-        </range>
-      </ray>
-      <plugin name="custom_dvl_plugin" filename="libfish_dvl_plugin.so"/>
-    </sensor>
-  </gazebo>
+  <!-- Fins -->
+  <xacro:fin_two_lines_macro
+      namespace="fish_hpurv"
+      parent_link="link_base"
+      fin_id="1"
+      min_joint_limit="-0.5"
+      max_joint_limit="0.5"
+      mesh_filename="$(find fish_hpurv)/meshes/link_caudal.stl"
+      fin_dynamics_time_constant="1.0"
+      fin_cross_section_area="0.1"
+      fluid_density="1000"
+      a0="0.0"
+      alpha_stall="15"
+      cla="0.1"
+      cla_stall="0.2"
+      cda="0.01"
+      cda_stall="0.02"
+      current_velocity_topic="/current_velocity">
+    <origin xyz="0.275 0 -0.02" rpy="1.57 3.14 0" />
+  </xacro:fin_two_lines_macro>
+  <xacro:fin_two_lines_macro
+      namespace="fish_hpurv"
+      parent_link="link_base"
+      fin_id="2"
+      min_joint_limit="-0.5"
+      max_joint_limit="0.5"
+      mesh_filename="$(find fish_hpurv)/meshes/link_pectoral_left.stl"
+      fin_dynamics_time_constant="1.0"
+      fin_cross_section_area="0.1"
+      fluid_density="1000"
+      a0="0.0"
+      alpha_stall="15"
+      cla="0.1"
+      cla_stall="0.2"
+      cda="0.01"
+      cda_stall="0.02"
+      current_velocity_topic="/current_velocity">
+    <origin xyz="0.25 0 0.045" rpy="-1.57 3.14 0" />
+  </xacro:fin_two_lines_macro>
+  <xacro:fin_two_lines_macro
+      namespace="fish_hpurv"
+      parent_link="link_base"
+      fin_id="3"
+      min_joint_limit="-0.5"
+      max_joint_limit="0.5"
+      mesh_filename="$(find fish_hpurv)/meshes/link_pectoral_right.stl"
+      fin_dynamics_time_constant="1.0"
+      fin_cross_section_area="0.1"
+      fluid_density="1000"
+      a0="0.0"
+      alpha_stall="15"
+      cla="0.1"
+      cla_stall="0.2"
+      cda="0.01"
+      cda_stall="0.02"
+      current_velocity_topic="/current_velocity">
+    <origin xyz="0.25 0 0.045" rpy="-1.57 3.14 0" />
+  </xacro:fin_two_lines_macro>
+  <!-- Gazebo plugins -->
   <gazebo>
     <plugin name="buoyancy_plugin" filename="libBuoyancyPlugin.so">
       <fluid_density>1000</fluid_density>
       <link name="link_base">
-        <volume>0.0122</volume>
-        <center_of_volume>0.0325815 0.0493006 0.02</center_of_volume>
-      </link>
-      <link name="link_caudal">
-        <volume>0.0002</volume>
-        <center_of_volume>-0.378805 0 -0.05</center_of_volume>
-      </link>
-      <link name="link_pectoral_left">
-        <volume>0.0001</volume>
-        <center_of_volume>0.0829833 -0.0470575 0.13</center_of_volume>
-      </link>
-      <link name="link_pectoral_right">
-        <volume>0.0001</volume>
-        <center_of_volume>0.0829833 0.0470575 0.13</center_of_volume>
+        <volume>0.001</volume>
+        <center_of_volume>0.246461 -0.269567 0.0980965</center_of_volume>
       </link>
       <link name="fish_hpurv/fin1">
         <volume>0.0000001</volume>
-        <center_of_volume>0.0829833 0.0470575 0.13</center_of_volume>
+        <center_of_volume>0 0 0</center_of_volume>
+      </link>
+      <link name="fish_hpurv/fin2">
+        <volume>0.0000001</volume>
+        <center_of_volume>0 0 0</center_of_volume>
+      </link>
+      <link name="fish_hpurv/fin3">
+        <volume>0.0000001</volume>
+        <center_of_volume>0 0 0</center_of_volume>
       </link>
     </plugin>
@@ -267,15 +113,15 @@
       <plugin>gazebo_ros2_control/GazeboSystem</plugin>
     </hardware>
-    <joint name="caudal_joint">
+    <joint name="fish_hpurv/fin1_joint">
       <command_interface name="position"/>
       <state_interface name="position"/>
       <state_interface name="velocity"/>
     </joint>
-    <joint name="joint1">
+    <joint name="fish_hpurv/fin2_joint">
       <command_interface name="position"/>
       <state_interface name="position"/>
       <state_interface name="velocity"/>
     </joint>
-    <joint name="joint2">
+    <joint name="fish_hpurv/fin3_joint">
       <command_interface name="position"/>
       <state_interface name="position"/>
@@ -283,22 +129,3 @@
     </joint>
   </ros2_control>
-<xacro:fin_two_lines_macro
-    namespace="fish_hpurv"
-    parent_link="link_base"
-    fin_id="1"
-    min_joint_limit="-0.5"
-    max_joint_limit="0.5"
-    mesh_filename="$(find fish_hpurv)/meshes/fin1.stl"
-    fin_dynamics_time_constant="1.0"
-    fin_cross_section_area="0.1"
-    fluid_density="1000"
-    a0="0.0"
-    alpha_stall="15"
-    cla="0.1"
-    cla_stall="0.2"
-    cda="0.01"
-    cda_stall="0.02"
-    current_velocity_topic="/current_velocity">
-  <origin xyz="0.1 0 0" rpy="0 0 0" />
-</xacro:fin_two_lines_macro>
 </robot>
